File: Micro.sch (KiCad schematic (older format))
At the start: 0 parts

Commit message: LPC + RAM + ROM Progress
Connections:
- no-connect marks 0 -> 1

Commit message: batch push
Connections:
- no-connect marks 1 -> 49
Changed lines of the file:
@@
 F0 "Power Supply" 50
 F1 "Power Suply.sch" 50
-F2 "IN_PWR_SUPPLY" I L 750 1350 50
 $EndSheet
 Wire Wire Line
@@
 Text Label 6400 4400 0    50   ~ 0
 SPIFI_SCK
-$Sheet
-S 8650 1150 1500 2650
-U 5F5DA166
-F0 "RAM" 50
-F1 "RAM.sch" 50
-F2 "A0" I L 8650 1250 50
-F3 "A1" I L 8650 1350 50
-F4 "A2" I L 8650 1450 50
-F5 "A3" I L 8650 1550 50
-F6 "A4" I L 8650 1650 50
-F7 "A5" I L 8650 1750 50
-F8 "A6" I L 8650 1850 50
-F9 "A7" I L 8650 1950 50
-F10 "A8" I L 8650 2050 50
-F11 "A9" I L 8650 2150 50
-F12 "A10" I L 8650 2250 50
-F13 "A11" I L 8650 2350 50
-F14 "A12" I L 8650 2450 50
-F15 "CS0" I L 8650 2600 50
-F16 "CKE" I L 8650 2800 50
-F17 "DQ0" I R 10150 1300 50
-F18 "DQ1" I R 10150 1400 50
-F19 "DQ2" I R 10150 1500 50
-F20 "DQ3" I R 10150 1600 50
-F21 "DQ4" I R 10150 1700 50
-F22 "DQ5" I R 10150 1800 50
-F23 "DQ6" I R 10150 1900 50
-F24 "DQ7" I R 10150 2000 50
-F25 "DQ8" I R 10150 2100 50
-F26 "DQ9" I R 10150 2200 50
-F27 "DQ10" I R 10150 2300 50
-F28 "DQ11" I R 10150 2400 50
-F29 "DQ12" I R 10150 2500 50
-F30 "DQ13" I R 10150 2600 50
-F31 "DQ14" I R 10150 2700 50
-F32 "DQ15" I R 10150 2800 50
-F33 "CLK" I L 8650 3200 50
-F34 "CS1" I L 8650 2700 50
-F35 "UDQM" I L 8650 3300 50
-F36 "LDQM" I L 8650 3400 50
-F37 "CAS#" I L 8650 3500 50
-F38 "RAS#" I L 8650 3600 50
-F39 "WE#" I L 8650 3700 50
-$EndSheet
 Wire Wire Line
 	5650 5900 6400 5900
@@
 	5650 2200 6400 2200
 Text Label 6400 2200 0    50   ~ 0
-EMC_A
+EMC_A7
 Wire Wire Line
 	5650 5800 6400 5800
@@
 Text Label 7900 2600 2    50   ~ 0
 EMC_DYCS0
-Wire Wire Line
-	5650 2500 6400 2500
 Text Label 7900 2700 2    50   ~ 0
 EMC_DYCS1
@@
 	10150 2800 10450 2800
 Wire Wire Line
-	6400 1750 5650 1750
-Text Label 6400 1750 0    50   ~ 0
-GPIO0[0]
-Wire Wire Line
 	7900 3300 8650 3300
 Wire Wire Line
@@
 Text Label 7900 3700 2    50   ~ 0
 EMC_WE
-Wire Wire Line
-	6400 1850 5650 1850
-Text Label 6400 1850 0    50   ~ 0
-GPIO0[1]
-Wire Wire Line
-	6400 3700 5650 3700
 Text Label 6400 2600 0    50   ~ 0
 EMC_WE
@@
 	6400 2600 5650 2600
 Wire Wire Line
-	3100 2550 3850 2550
-Text Label 3100 2550 2    50   ~ 0
-EMC_CKEOUT0
+	3100 1650 3850 1650
+Text Label 3100 1650 2    50   ~ 0
+EMC_CKEOUT1
 Wire Wire Line
 	3100 2350 3850 2350
@@
 Text Label 7900 3300 2    50   ~ 0
 EMC_BLS0
+$Sheet
+S 8650 1150 1500 2650
+U 5F5DA166
+F0 "RAM" 50
+F1 "RAM.sch" 50
+F2 "A0" I L 8650 1250 50
+F3 "A1" I L 8650 1350 50
+F4 "A2" I L 8650 1450 50
+F5 "A3" I L 8650 1550 50
+F6 "A4" I L 8650 1650 50
+F7 "A5" I L 8650 1750 50
+F8 "A6" I L 8650 1850 50
+F9 "A7" I L 8650 1950 50
+F10 "A8" I L 8650 2050 50
+F11 "A9" I L 8650 2150 50
+F12 "A10" I L 8650 2250 50
+F13 "A11" I L 8650 2350 50
+F14 "A12" I L 8650 2450 50
+F15 "CS0" I L 8650 2600 50
+F16 "DQ0" I R 10150 1300 50
+F17 "DQ1" I R 10150 1400 50
+F18 "DQ2" I R 10150 1500 50
+F19 "DQ3" I R 10150 1600 50
+F20 "DQ4" I R 10150 1700 50
+F21 "DQ5" I R 10150 1800 50
+F22 "DQ6" I R 10150 1900 50
+F23 "DQ7" I R 10150 2000 50
+F24 "DQ8" I R 10150 2100 50
+F25 "DQ9" I R 10150 2200 50
+F26 "DQ10" I R 10150 2300 50
+F27 "DQ11" I R 10150 2400 50
+F28 "DQ12" I R 10150 2500 50
+F29 "DQ13" I R 10150 2600 50
+F30 "DQ14" I R 10150 2700 50
+F31 "DQ15" I R 10150 2800 50
+F32 "CLK" I L 8650 3200 50
+F33 "CS1" I L 8650 2700 50
+F34 "UDQM" I L 8650 3300 50
+F35 "LDQM" I L 8650 3400 50
+F36 "CAS#" I L 8650 3500 50
+F37 "RAS#" I L 8650 3600 50
+F38 "WE#" I L 8650 3700 50
+F39 "CKE0" I L 8650 2800 50
+F40 "CKE1" I L 8650 2900 50
+$EndSheet
+NoConn ~ 3850 2450
+NoConn ~ 3850 2650
+NoConn ~ 3850 2750
+NoConn ~ 3850 2850
+NoConn ~ 3850 2950
+NoConn ~ 3850 3050
+NoConn ~ 3850 3150
+NoConn ~ 3850 3250
+NoConn ~ 3850 3350
+NoConn ~ 3850 3450
+NoConn ~ 3850 3550
+NoConn ~ 3850 3650
+NoConn ~ 3850 3750
+NoConn ~ 3850 3850
+NoConn ~ 3850 3950
+NoConn ~ 3850 4050
+NoConn ~ 3850 4150
+NoConn ~ 3850 4250
+NoConn ~ 3850 4350
+NoConn ~ 3850 4450
+NoConn ~ 3850 4550
+NoConn ~ 3850 4650
+NoConn ~ 3850 4750
+NoConn ~ 5650 4100
+NoConn ~ 5650 4200
+NoConn ~ 5650 4300
+NoConn ~ 5650 5300
+NoConn ~ 5650 5400
+NoConn ~ 5650 5500
+NoConn ~ 5650 6450
+NoConn ~ 5650 6550
+NoConn ~ 5650 6650
+NoConn ~ 5650 6750
+NoConn ~ 5650 6850
+NoConn ~ 5650 6950
+NoConn ~ 5650 7050
+NoConn ~ 5650 7150
+NoConn ~ 5650 1750
+NoConn ~ 5650 1850
+NoConn ~ 5650 2500
+NoConn ~ 5650 3700
+NoConn ~ 3850 1450
+NoConn ~ 3850 1750
+NoConn ~ 5650 3900
+NoConn ~ 6400 5000
+NoConn ~ 6400 2300
+NoConn ~ 3100 2250
+NoConn ~ 3100 2150
+Wire Wire Line
+	3100 2550 3850 2550
+Text Label 3100 2550 2    50   ~ 0
+EMC_CKEOUT0
 $EndSCHEMATC
