File: Power Suply.sch (KiCad schematic (older format))
At the start: 7 parts

Commit message: batch push
Parts:
- added J1: Barrel_Jack, symbol Connector:Barrel_Jack
- gave numbers to parts that had none: 7
Connections:
- net GND: now also J1.2
- net IN_PWR_SUPPLY renamed Vin
- net Vin: now also J1.1
Changed lines of the file:
@@
 $Descr A4 11693 8268
 encoding utf-8
-Sheet 5 7
+Sheet 3 7
 Title ""
 Date ""
@@
 Comment4 ""
 $EndDescr
-Text HLabel 1850 1350 0    50   Input ~ 0
-IN_PWR_SUPPLY
-$Comp
-L Regulator_Switching:LM2576HVS-5 U?
+$Comp
+L Regulator_Switching:LM2576HVS-5 U3
 U 1 1 5F10E5BA
 P 3350 1450
-F 0 "U?" H 3350 1817 50  0000 C CNN
+F 0 "U3" H 3350 1817 50  0000 C CNN
 F 1 "LM2576HVS-5" H 3350 1726 50  0000 C CNN
 F 2 "Package_TO_SOT_SMD:TO-263-5_TabPin3" H 3350 1200 50  0001 L CIN
@@
 $EndComp
 $Comp
-L power:GND #PWR?
+L power:GND #PWR010
 U 1 1 5F10F4A6
 P 2850 1750
-F 0 "#PWR?" H 2850 1500 50  0001 C CNN
+F 0 "#PWR010" H 2850 1500 50  0001 C CNN
 F 1 "GND" H 2855 1577 50  0000 C CNN
 F 2 "" H 2850 1750 50  0001 C CNN
@@
 $EndComp
 $Comp
-L power:GND #PWR?
+L power:GND #PWR012
 U 1 1 5F10F901
 P 3350 1750
-F 0 "#PWR?" H 3350 1500 50  0001 C CNN
+F 0 "#PWR012" H 3350 1500 50  0001 C CNN
 F 1 "GND" H 3355 1577 50  0000 C CNN
 F 2 "" H 3350 1750 50  0001 C CNN
@@
 $EndComp
 $Comp
-L Device:CP C?
+L Device:CP C16
 U 1 1 5F10FE25
 P 5250 1700
-F 0 "C?" H 5368 1746 50  0000 L CNN
+F 0 "C16" H 5368 1746 50  0000 L CNN
 F 1 "1000u" H 5368 1655 50  0000 L CNN
 F 2 "Capacitor_Tantalum_SMD:CP_EIA-1608-08_AVX-J" H 5288 1550 50  0001 C CNN
@@
 $EndComp
 $Comp
-L pspice:INDUCTOR L?
+L pspice:INDUCTOR L1
 U 1 1 5F112663
 P 4650 1550
-F 0 "L?" H 4650 1450 50  0000 C CNN
+F 0 "L1" H 4650 1450 50  0000 C CNN
 F 1 "100uH" H 4650 1674 50  0000 C CNN
 F 2 "Inductor_SMD:L_12x12mm_H6mm" H 4650 1550 50  0001 C CNN
@@
 	4900 1550 5250 1550
 $Comp
-L power:GND #PWR?
+L power:GND #PWR015
 U 1 1 5F11485F
 P 4100 1850
-F 0 "#PWR?" H 4100 1600 50  0001 C CNN
+F 0 "#PWR015" H 4100 1600 50  0001 C CNN
 F 1 "GND" H 4105 1677 50  0000 C CNN
 F 2 "" H 4100 1850 50  0001 C CNN
@@
 $EndComp
 $Comp
-L power:GND #PWR?
+L power:GND #PWR016
 U 1 1 5F114BCD
 P 5250 1850
-F 0 "#PWR?" H 5250 1600 50  0001 C CNN
+F 0 "#PWR016" H 5250 1600 50  0001 C CNN
 F 1 "GND" H 5255 1677 50  0000 C CNN
 F 2 "" H 5250 1850 50  0001 C CNN
@@
 	2450 1350 2850 1350
 $Comp
-L power:GND #PWR?
+L power:GND #PWR08
 U 1 1 5F117364
 P 2450 1750
-F 0 "#PWR?" H 2450 1500 50  0001 C CNN
+F 0 "#PWR08" H 2450 1500 50  0001 C CNN
 F 1 "GND" H 2455 1577 50  0000 C CNN
 F 2 "" H 2450 1750 50  0001 C CNN
@@
 	3850 1550 4100 1550
 $Comp
-L Device:D_Schottky D?
+L Device:D_Schottky D1
 U 1 1 5F129415
 P 4100 1700
-F 0 "D?" V 4054 1780 50  0000 L CNN
+F 0 "D1" V 4054 1780 50  0000 L CNN
 F 1 "D_Schottky" V 4145 1780 50  0000 L CNN
 F 2 "Diode_SMD:D_SMC" H 4100 1700 50  0001 C CNN
@@
 	4100 1550 4400 1550
 $Comp
-L Device:CP C?
+L Device:CP C14
 U 1 1 5F11735B
 P 2450 1500
-F 0 "C?" H 2568 1546 50  0000 L CNN
+F 0 "C14" H 2568 1546 50  0000 L CNN
 F 1 "100uF" H 2568 1455 50  0000 L CNN
 F 2 "Capacitor_Tantalum_SMD:CP_EIA-1608-08_AVX-J" H 2488 1350 50  0001 C CNN
@@
 Connection ~ 5250 1350
 $Comp
-L power:PWR_FLAG #FLG?
+L power:PWR_FLAG #FLG01
 U 1 1 5F12E9B1
 P 2100 1350
-F 0 "#FLG?" H 2100 1425 50  0001 C CNN
+F 0 "#FLG01" H 2100 1425 50  0001 C CNN
 F 1 "PWR_FLAG" H 2100 1523 50  0000 C CNN
 F 2 "" H 2100 1350 50  0001 C CNN
@@
 $EndComp
 Connection ~ 2100 1350
-Wire Wire Line
-	2100 1350 1850 1350
-$Comp
-L power:PWR_FLAG #FLG?
+$Comp
+L power:PWR_FLAG #FLG02
 U 1 1 5F12F184
 P 2100 1800
-F 0 "#FLG?" H 2100 1875 50  0001 C CNN
+F 0 "#FLG02" H 2100 1875 50  0001 C CNN
 F 1 "PWR_FLAG" H 2100 1973 50  0000 C CNN
 F 2 "" H 2100 1800 50  0001 C CNN
@@
 $EndComp
 $Comp
-L power:GND #PWR?
+L power:GND #PWR07
 U 1 1 5F131C10
 P 2100 1800
-F 0 "#PWR?" H 2100 1550 50  0001 C CNN
+F 0 "#PWR07" H 2100 1550 50  0001 C CNN
 F 1 "GND" H 2105 1627 50  0000 C CNN
 F 2 "" H 2100 1800 50  0001 C CNN
@@
 $EndComp
 $Comp
-L power:+5V #PWR?
+L power:+5V #PWR017
 U 1 1 5F1CB9C0
 P 5800 1350
-F 0 "#PWR?" H 5800 1200 50  0001 C CNN
+F 0 "#PWR017" H 5800 1200 50  0001 C CNN
 F 1 "+5V" H 5815 1523 50  0000 C CNN
 F 2 "" H 5800 1350 50  0001 C CNN
@@
 $EndComp
 $Comp
-L Regulator_Linear:LM117_TO3 U?
+L Regulator_Linear:LM117_TO3 U2
 U 1 1 5F1CC8F8
 P 3100 3200
-F 0 "U?" H 3100 3442 50  0000 C CNN
+F 0 "U2" H 3100 3442 50  0000 C CNN
 F 1 "LM117_TO3" H 3100 3351 50  0000 C CNN
 F 2 "Package_TO_SOT_SMD:SOT-223-3_TabPin2" H 3100 3400 50  0001 C CIN
@@
 $EndComp
 $Comp
-L power:+5V #PWR?
+L power:+5V #PWR09
 U 1 1 5F1CCE6F
 P 2800 3200
-F 0 "#PWR?" H 2800 3050 50  0001 C CNN
+F 0 "#PWR09" H 2800 3050 50  0001 C CNN
 F 1 "+5V" H 2815 3373 50  0000 C CNN
 F 2 "" H 2800 3200 50  0001 C CNN
@@
 $EndComp
 $Comp
-L power:GND #PWR?
+L power:GND #PWR011
 U 1 1 5F1CD19C
 P 3100 3500
-F 0 "#PWR?" H 3100 3250 50  0001 C CNN
+F 0 "#PWR011" H 3100 3250 50  0001 C CNN
 F 1 "GND" H 3105 3327 50  0000 C CNN
 F 2 "" H 3100 3500 50  0001 C CNN
@@
 	3650 3200 3650 3350
 $Comp
-L Device:CP C?
+L Device:CP C15
 U 1 1 5F1CDFCB
 P 3650 3500
-F 0 "C?" H 3768 3546 50  0000 L CNN
+F 0 "C15" H 3768 3546 50  0000 L CNN
 F 1 "100u" H 3768 3455 50  0000 L CNN
 F 2 "Capacitor_Tantalum_SMD:CP_EIA-1608-08_AVX-J" H 3688 3350 50  0001 C CNN
@@
 $EndComp
 $Comp
-L power:GND #PWR?
+L power:GND #PWR014
 U 1 1 5F1CE4A9
 P 3650 3650
-F 0 "#PWR?" H 3650 3400 50  0001 C CNN
+F 0 "#PWR014" H 3650 3400 50  0001 C CNN
 F 1 "GND" H 3655 3477 50  0000 C CNN
 F 2 "" H 3650 3650 50  0001 C CNN
@@
 $EndComp
 $Comp
-L power:+3.3V #PWR?
+L power:+3.3V #PWR013
 U 1 1 5F1CEA2F
 P 3650 3200
-F 0 "#PWR?" H 3650 3050 50  0001 C CNN
+F 0 "#PWR013" H 3650 3050 50  0001 C CNN
 F 1 "+3.3V" H 3665 3373 50  0000 C CNN
 F 2 "" H 3650 3200 50  0001 C CNN
@@
 Text Notes 6000 3900 0    50   ~ 0
 O: 3V
+$Comp
+L Connector:Barrel_Jack J1
+U 1 1 5FE17B5C
+P 1300 1600
+F 0 "J1" H 1357 1925 50  0000 C CNN
+F 1 "Barrel_Jack" H 1350 1400 50  0000 C CNN
+F 2 "" H 1350 1560 50  0001 C CNN
+F 3 "~" H 1350 1560 50  0001 C CNN
+	1    1300 1600
+	1    0    0    -1
+$EndComp
+Wire Wire Line
+	1600 1500 1600 1350
+Wire Wire Line
+	1600 1350 2100 1350
+Wire Wire Line
+	1600 1700 1600 1800
+Wire Wire Line
+	1600 1800 2100 1800
+Connection ~ 2100 1800
+$Comp
+L power:PWR_FLAG #FLG0102
+U 1 1 5FE26BE5
+P 5250 1350
+F 0 "#FLG0102" H 5250 1425 50  0001 C CNN
+F 1 "PWR_FLAG" H 5250 1523 50  0000 C CNN
+F 2 "" H 5250 1350 50  0001 C CNN
+F 3 "~" H 5250 1350 50  0001 C CNN
+	1    5250 1350
+	1    0    0    -1
+$EndComp
 $EndSCHEMATC
