File: ROM.sch (KiCad schematic (older format))
At the start: 1 part

Commit message: batch push
Parts:
- gave numbers to parts that had none: 1
Changed lines of the file:
@@
 AR Path="/5F64163B/5F8EEAF3/5F8F800A" Ref="NOR_FLASH?"  Part="1"
 AR Path="/5F64163B/5F8EEAFB/5F8F800A" Ref="NOR_FLASH?"  Part="1"
-AR Path="/5F64163B/5F8F800A" Ref="NOR_FLASH?"  Part="1"
-F 0 "NOR_FLASH?" H 5150 1765 50  0000 C CNN
+AR Path="/5F64163B/5F8F800A" Ref="NOR_FLASH1"  Part="1"
+F 0 "NOR_FLASH1" H 5150 1765 50  0000 C CNN
 F 1 "NOR_FLASH-Micron-N25Q064A" H 5150 1674 50  0000 C CNN
 F 2 "" H 4750 1600 50  0001 C CNN
@@
 AR Path="/5F64163B/5F8EEAF3/5F8F801A" Ref="#PWR?"  Part="1"
 AR Path="/5F64163B/5F8EEAFB/5F8F801A" Ref="#PWR?"  Part="1"
-AR Path="/5F64163B/5F8F801A" Ref="#PWR?"  Part="1"
-F 0 "#PWR?" H 3800 1700 50  0001 C CNN
+AR Path="/5F64163B/5F8F801A" Ref="#PWR018"  Part="1"
+F 0 "#PWR018" H 3800 1700 50  0001 C CNN
 F 1 "+3V3" H 3815 2023 50  0000 C CNN
 F 2 "" H 3800 1850 50  0001 C CNN
@@
 AR Path="/5F64163B/5F8EEAF3/5F8F8022" Ref="#PWR?"  Part="1"
 AR Path="/5F64163B/5F8EEAFB/5F8F8022" Ref="#PWR?"  Part="1"
-AR Path="/5F64163B/5F8F8022" Ref="#PWR?"  Part="1"
-F 0 "#PWR?" H 6550 2150 50  0001 C CNN
+AR Path="/5F64163B/5F8F8022" Ref="#PWR019"  Part="1"
+F 0 "#PWR019" H 6550 2150 50  0001 C CNN
 F 1 "GND" H 6555 2227 50  0000 C CNN
 F 2 "" H 6550 2400 50  0001 C CNN
