File: MICRO-LPC4337JBD144.sch (KiCad schematic (older format))
At the start: 16 parts

Commit message: LPC + ROM + RAM sch
Parts:
- R?: value R -> 100K
- U?: symbol LPC4337JBD144:LPC4337JBD144 -> Micro-rescue:LPC4337JBD144-LPC4337JBD144
Connections:
- net labels added: CLK0, CLK2, P0_0, P0_1, P1_0, P1_1, P1_10, P1_11, P1_12, P1_13, P1_14, P1_15, P1_16, P1_17, P1_18, P1_19, P1_2, P1_20, P1_3, P1_4, P1_5, P1_6, P1_7, P1_8, P1_9, P2_0, P2_1, P2_10, P2_11, P2_12, P2_13, P2_2, P2_3, P2_4, P2_5, P2_6, P2_7, P2_8, P2_9, P3_0, P3_1, P3_2, P3_3, P3_4, P3_5, P3_6, P3_7, P3_8, P4_0, P4_1, P4_10, P4_2, P4_3, P4_4, P4_5, P4_6, P4_7, P4_8, P4_9, P5_0, P5_1, P5_2, P5_3, P5_4, P5_5, P5_6, P5_7, P6_0, P6_1, P6_10, P6_11, P6_12, P6_2, P6_3, P6_4, P6_5, P6_6, P6_7, P6_8, P6_9, P7_0, P7_1, P7_2, P7_3, P7_4, P7_5, P7_6, P7_7, P9_5, P9_6
- wire segments 79 -> 169

Commit message: batch push
Parts:
- gave numbers to parts that had none: 16
Connections:
- no-connect marks 9 -> 35
Changed lines of the file:
@@
 Comment4 ""
 $EndDescr
-$Comp
-L Micro-rescue:LPC4337JBD144-LPC4337JBD144 U?
-U 1 1 5F5DA26E
-P 4550 2500
-AR Path="/5F5DA26E" Ref="U?"  Part="1"
-AR Path="/5F5D97EE/5F5DA26E" Ref="U?"  Part="1"
-F 0 "U?" V 3850 -650 60  0000 R CNN
-F 1 "LPC4337JBD144" V 3700 -550 60  0000 R CNN
-F 2 "" H 4450 6450 60  0000 C CNN
-F 3 "" H 4450 6450 60  0000 C CNN
-	1    4550 2500
-	0    1    1    0
-$EndComp
 Connection ~ 1400 2600
 Wire Wire Line
@@
 	1200 2500 1200 2600
 $Comp
-L power:GND #PWR?
+L power:GND #PWR01
 U 1 1 5F603909
 P 1200 2600
-F 0 "#PWR?" H 1200 2350 50  0001 C CNN
+F 0 "#PWR01" H 1200 2350 50  0001 C CNN
 F 1 "GND" H 1205 2427 50  0000 C CNN
 F 2 "" H 1200 2600 50  0001 C CNN
@@
 	9700 3300 9700 3450
 $Comp
-L Device:C C?
+L Device:C C2
 U 1 1 5F5DEC74
 P 10100 2050
-F 0 "C?" V 10000 1950 50  0000 C CNN
+F 0 "C2" V 10000 1950 50  0000 C CNN
 F 1 "100nF" V 10000 2150 50  0000 C CNN
 F 2 "" H 10138 1900 50  0001 C CNN
@@
 $EndComp
 $Comp
-L Device:C C?
+L Device:C C3
 U 1 1 5F5E01AD
 P 10100 2250
-F 0 "C?" V 10000 2150 50  0000 C CNN
+F 0 "C3" V 10000 2150 50  0000 C CNN
 F 1 "100nF" V 10000 2350 50  0000 C CNN
 F 2 "" H 10138 2100 50  0001 C CNN
@@
 $EndComp
 $Comp
-L Device:C C?
+L Device:C C4
 U 1 1 5F5E06F3
 P 10100 2450
-F 0 "C?" V 10000 2350 50  0000 C CNN
+F 0 "C4" V 10000 2350 50  0000 C CNN
 F 1 "100nF" V 10000 2550 50  0000 C CNN
 F 2 "" H 10138 2300 50  0001 C CNN
@@
 $EndComp
 $Comp
-L Device:C C?
+L Device:C C5
 U 1 1 5F5E0B15
 P 10100 2650
-F 0 "C?" V 10000 2550 50  0000 C CNN
+F 0 "C5" V 10000 2550 50  0000 C CNN
 F 1 "100nF" V 10000 2750 50  0000 C CNN
 F 2 "" H 10138 2500 50  0001 C CNN
@@
 $EndComp
 $Comp
-L Device:C C?
+L Device:C C6
 U 1 1 5F5E102B
 P 10100 2850
-F 0 "C?" V 10000 2750 50  0000 C CNN
+F 0 "C6" V 10000 2750 50  0000 C CNN
 F 1 "100nF" V 10000 2950 50  0000 C CNN
 F 2 "" H 10138 2700 50  0001 C CNN
@@
 $EndComp
 $Comp
-L Device:C C?
+L Device:C C7
 U 1 1 5F5E2381
 P 10100 3050
-F 0 "C?" V 10000 2950 50  0000 C CNN
+F 0 "C7" V 10000 2950 50  0000 C CNN
 F 1 "100nF" V 10000 3150 50  0000 C CNN
 F 2 "" H 10138 2900 50  0001 C CNN
@@
 	9700 3050 9700 3100
 $Comp
-L Device:C C?
+L Device:C C8
 U 1 1 5F5F26A3
 P 10100 3250
-F 0 "C?" V 10000 3150 50  0000 C CNN
+F 0 "C8" V 10000 3150 50  0000 C CNN
 F 1 "100nF" V 10000 3350 50  0000 C CNN
 F 2 "" H 10138 3100 50  0001 C CNN
@@
 $EndComp
 $Comp
-L Device:C C?
+L Device:C C9
 U 1 1 5F5F26AD
 P 10100 3450
-F 0 "C?" V 10000 3350 50  0000 C CNN
+F 0 "C9" V 10000 3350 50  0000 C CNN
 F 1 "100nF" V 10000 3550 50  0000 C CNN
 F 2 "" H 10138 3300 50  0001 C CNN
@@
 $EndComp
 $Comp
-L Device:C C?
+L Device:C C10
 U 1 1 5F5F26B7
 P 10100 3650
-F 0 "C?" V 10000 3550 50  0000 C CNN
+F 0 "C10" V 10000 3550 50  0000 C CNN
 F 1 "100nF" V 10000 3750 50  0000 C CNN
 F 2 "" H 10138 3500 50  0001 C CNN
@@
 $EndComp
 $Comp
-L Device:C C?
+L Device:C C11
 U 1 1 5F5F26C1
 P 10100 3850
-F 0 "C?" V 10000 3750 50  0000 C CNN
+F 0 "C11" V 10000 3750 50  0000 C CNN
 F 1 "100nF" V 10000 3950 50  0000 C CNN
 F 2 "" H 10138 3700 50  0001 C CNN
@@
 $EndComp
 $Comp
-L Device:C C?
+L Device:C C12
 U 1 1 5F5F26CB
 P 10100 4050
-F 0 "C?" V 10000 3950 50  0000 C CNN
+F 0 "C12" V 10000 3950 50  0000 C CNN
 F 1 "100nF" V 10000 4150 50  0000 C CNN
 F 2 "" H 10138 3900 50  0001 C CNN
@@
 $EndComp
 $Comp
-L Device:C C?
+L Device:C C13
 U 1 1 5F5F26D5
 P 10100 4250
-F 0 "C?" V 10000 4150 50  0000 C CNN
+F 0 "C13" V 10000 4150 50  0000 C CNN
 F 1 "100nF" V 10000 4350 50  0000 C CNN
 F 2 "" H 10138 4100 50  0001 C CNN
@@
 	10500 3100 10500 2950
 $Comp
-L power:GND #PWR?
+L power:GND #PWR06
 U 1 1 5F608AE0
 P 10500 3100
-F 0 "#PWR?" H 10500 2850 50  0001 C CNN
+F 0 "#PWR06" H 10500 2850 50  0001 C CNN
 F 1 "GND" H 10505 2927 50  0000 C CNN
 F 2 "" H 10500 3100 50  0001 C CNN
@@
 Connection ~ 9700 2050
 $Comp
-L power:+3.3V #PWR?
+L power:+3.3V #PWR05
 U 1 1 5F60BEE1
 P 9700 1850
-F 0 "#PWR?" H 9700 1700 50  0001 C CNN
+F 0 "#PWR05" H 9700 1700 50  0001 C CNN
 F 1 "+3.3V" H 9715 2023 50  0000 C CNN
 F 2 "" H 9700 1850 50  0001 C CNN
@@
 NoConn ~ 9150 1550
 $Comp
-L Switch:SW_Push_Dual_x2 SW?
+L Switch:SW_Push_Dual_x2 SW1
 U 1 1 5F61A5A7
 P 3950 5450
-F 0 "SW?" V 3904 5598 50  0000 L CNN
+F 0 "SW1" V 3904 5598 50  0000 L CNN
 F 1 "SW_Push_Dual_x2" V 3995 5598 50  0000 L CNN
 F 2 "" H 3950 5650 50  0001 C CNN
@@
 	3950 5650 3950 5750
 $Comp
-L power:GND #PWR?
+L power:GND #PWR04
 U 1 1 5F61D171
 P 3950 5800
-F 0 "#PWR?" H 3950 5550 50  0001 C CNN
+F 0 "#PWR04" H 3950 5550 50  0001 C CNN
 F 1 "GND" H 3955 5627 50  0000 C CNN
 F 2 "" H 3950 5800 50  0001 C CNN
@@
 $EndComp
 $Comp
-L Device:R R?
+L Device:R R1
 U 1 1 5F61DCD4
 P 3300 5400
-F 0 "R?" H 3370 5446 50  0000 L CNN
+F 0 "R1" H 3370 5446 50  0000 L CNN
 F 1 "100K" V 3300 5300 50  0000 L CNN
 F 2 "" V 3230 5400 50  0001 C CNN
@@
 $EndComp
 $Comp
-L power:+3.3V #PWR?
+L power:+3.3V #PWR03
 U 1 1 5F6200AA
 P 3300 5850
-F 0 "#PWR?" H 3300 5700 50  0001 C CNN
+F 0 "#PWR03" H 3300 5700 50  0001 C CNN
 F 1 "+3.3V" H 3315 6023 50  0000 C CNN
 F 2 "" H 3300 5850 50  0001 C CNN
@@
 	3300 5850 3300 5550
 $Comp
-L Device:C C?
+L Device:C C1
 U 1 1 5F63065B
 P 3600 5400
-F 0 "C?" H 3715 5446 50  0000 L CNN
+F 0 "C1" H 3715 5446 50  0000 L CNN
 F 1 "C" H 3715 5355 50  0000 L CNN
 F 2 "" H 3638 5250 50  0001 C CNN
@@
 	1200 2900 1400 2900
 $Comp
-L power:GNDA #PWR?
+L power:GNDA #PWR02
 U 1 1 5F643716
 P 1200 3000
-F 0 "#PWR?" H 1200 2750 50  0001 C CNN
+F 0 "#PWR02" H 1200 2750 50  0001 C CNN
 F 1 "GNDA" H 1205 2827 50  0000 C CNN
 F 2 "" H 1200 3000 50  0001 C CNN
@@
 Wire Wire Line
 	8900 1550 8900 1400
-Text HLabel 8900 1400 1    50   Input ~ 0
+Text HLabel 8900 1400 1    50   Output ~ 0
 P0_0
 Wire Wire Line
@@
 Wire Wire Line
 	8350 1400 8350 1550
-Text HLabel 8250 1400 1    50   Input ~ 0
+Text HLabel 8250 1400 1    50   Output ~ 0
 P1_4
 Wire Wire Line
@@
 Text HLabel 6050 4400 3    50   Input ~ 0
 P9_6
+NoConn ~ 2200 1550
+NoConn ~ 2300 1550
+NoConn ~ 2500 1550
+NoConn ~ 2600 1550
+NoConn ~ 2750 1550
+NoConn ~ 2850 1550
+NoConn ~ 2950 1550
+NoConn ~ 5900 4250
+NoConn ~ 5500 4250
+NoConn ~ 5400 4250
+NoConn ~ 5300 4250
+NoConn ~ 5200 4250
+NoConn ~ 5100 4250
+NoConn ~ 5000 4250
+NoConn ~ 4800 4250
+NoConn ~ 4700 4250
+NoConn ~ 4600 4250
+NoConn ~ 4500 4250
+NoConn ~ 4400 4250
+NoConn ~ 4200 4250
+NoConn ~ 4100 4250
+NoConn ~ 3900 4250
+NoConn ~ 3800 4250
+NoConn ~ 1400 3100
+NoConn ~ 1400 3300
+$Comp
+L Micro-rescue:LPC4337JBD144-LPC4337JBD144 U?
+U 1 1 5F5DA26E
+P 4550 2500
+AR Path="/5F5DA26E" Ref="U?"  Part="1"
+AR Path="/5F5D97EE/5F5DA26E" Ref="U1"  Part="1"
+F 0 "U1" V 4897 -694 60  0000 R CNN
+F 1 "LPC4337JBD144" V 5003 -694 60  0000 R CNN
+F 2 "" H 4450 6450 60  0000 C CNN
+F 3 "" H 4450 6450 60  0000 C CNN
+	1    4550 2500
+	0    1    1    0
+$EndComp
+$Comp
+L power:PWR_FLAG #FLG0101
+U 1 1 5FE22055
+P 1200 2900
+F 0 "#FLG0101" H 1200 2975 50  0001 C CNN
+F 1 "PWR_FLAG" H 1200 3073 50  0000 C CNN
+F 2 "" H 1200 2900 50  0001 C CNN
+F 3 "~" H 1200 2900 50  0001 C CNN
+	1    1200 2900
+	1    0    0    -1
+$EndComp
+Connection ~ 1200 2900
+NoConn ~ 3450 4250
 $EndSCHEMATC

Commit message: Added XTALs, Removed WIP Initialization and Added NPXLPCOPEN
Parts:
- added C17, C18, C19, C20: C, symbol Device:C
- added R2, R3: 10M, symbol Device:R
- added Y1: 12MHz, symbol Device:Crystal_GND24
- added Y2: 32.768K, symbol Device:Crystal_GND24
Connections:
- net GND: now also C17.2, C18.2, C19.2, C20.2, Y1.2, Y1.4
- net XTAL1: now reaches U1.12 (XTAL1)
- net XTAL1: now also U1.13 (XTAL2), C17.1, C18.1, R2.1, R2.2, Y1.1, Y1.3
- net RTCX1: now reaches U1.125 (RTCX1)
- net RTCX1: now also U1.126 (RTCX2), C19.1, C20.1, R3.1, R3.2, Y2.1, Y2.3
- no-connect marks 35 -> 33
Changed lines of the file:
@@
 Comment4 ""
 $EndDescr
-Connection ~ 1400 2600
-Wire Wire Line
-	1400 2600 1400 2500
-Connection ~ 1400 2700
-Wire Wire Line
-	1400 2700 1400 2600
-Wire Wire Line
-	1400 2800 1400 2700
 Wire Wire Line
 	1400 2500 1200 2500
@@
 Wire Wire Line
 	3600 4250 3600 5250
-Connection ~ 1400 2500
 Wire Wire Line
 	1200 3000 1200 2900
@@
 NoConn ~ 2200 1550
 NoConn ~ 2300 1550
-NoConn ~ 2500 1550
-NoConn ~ 2600 1550
-NoConn ~ 2750 1550
-NoConn ~ 2850 1550
 NoConn ~ 2950 1550
 NoConn ~ 5900 4250
@@
 NoConn ~ 1400 3300
 $Comp
+L power:PWR_FLAG #FLG0101
+U 1 1 5FE22055
+P 1200 2900
+F 0 "#FLG0101" H 1200 2975 50  0001 C CNN
+F 1 "PWR_FLAG" H 1200 3073 50  0000 C CNN
+F 2 "" H 1200 2900 50  0001 C CNN
+F 3 "~" H 1200 2900 50  0001 C CNN
+	1    1200 2900
+	1    0    0    -1
+$EndComp
+Connection ~ 1200 2900
+NoConn ~ 3450 4250
+$Comp
+L Device:Crystal_GND24 Y2
+U 1 1 5F7DF11D
+P 1250 6200
+F 0 "Y2" V 850 6150 50  0000 L CNN
+F 1 "32.768K" V 950 6100 50  0000 L CNN
+F 2 "" H 1250 6200 50  0001 C CNN
+F 3 "~" H 1250 6200 50  0001 C CNN
+	1    1250 6200
+	0    1    1    0
+$EndComp
+Wire Wire Line
+	1250 6050 1900 6050
+Wire Wire Line
+	1900 6050 1900 6350
+$Comp
+L power:GND #PWR0101
+U 1 1 5F807DC0
+P 850 6200
+F 0 "#PWR0101" H 850 5950 50  0001 C CNN
+F 1 "GND" V 855 6072 50  0000 R CNN
+F 2 "" H 850 6200 50  0001 C CNN
+F 3 "" H 850 6200 50  0001 C CNN
+	1    850  6200
+	0    1    1    0
+$EndComp
+$Comp
+L Device:R R3
+U 1 1 5F84114A
+P 2100 6200
+F 0 "R3" H 2170 6246 50  0000 L CNN
+F 1 "10M" H 2170 6155 50  0000 L CNN
+F 2 "" V 2030 6200 50  0001 C CNN
+F 3 "~" H 2100 6200 50  0001 C CNN
+	1    2100 6200
+	1    0    0    -1
+$EndComp
+Wire Wire Line
+	2100 6050 1900 6050
+Connection ~ 1900 6050
+Wire Wire Line
+	2100 6350 1900 6350
+Connection ~ 1900 6350
+Wire Wire Line
+	2100 6050 2450 6050
+Connection ~ 2100 6050
+Wire Wire Line
+	2100 6350 2450 6350
+Connection ~ 2100 6350
+Wire Wire Line
+	1250 6050 1150 6050
+Wire Wire Line
+	850  6050 850  6200
+Connection ~ 1250 6050
+Connection ~ 850  6200
+Wire Wire Line
+	850  6200 850  6350
+$Comp
+L Device:C C19
+U 1 1 5F899E7D
+P 1000 6050
+F 0 "C19" V 748 6050 50  0000 C CNN
+F 1 "C" V 839 6050 50  0000 C CNN
+F 2 "" H 1038 5900 50  0001 C CNN
+F 3 "~" H 1000 6050 50  0001 C CNN
+	1    1000 6050
+	0    1    1    0
+$EndComp
+$Comp
+L Device:C C20
+U 1 1 5F89B81A
+P 1000 6350
+F 0 "C20" V 1300 6350 50  0000 C CNN
+F 1 "C" V 1200 6350 50  0000 C CNN
+F 2 "" H 1038 6200 50  0001 C CNN
+F 3 "~" H 1000 6350 50  0001 C CNN
+	1    1000 6350
+	0    1    1    0
+$EndComp
+Connection ~ 1250 6350
+Wire Wire Line
+	1900 6350 1250 6350
+Wire Wire Line
+	1150 6350 1250 6350
+$Comp
+L Device:Crystal_GND24 Y1
+U 1 1 5F8E2472
+P 1200 7100
+F 0 "Y1" V 800 7050 50  0000 L CNN
+F 1 "12MHz" V 900 7000 50  0000 L CNN
+F 2 "" H 1200 7100 50  0001 C CNN
+F 3 "~" H 1200 7100 50  0001 C CNN
+	1    1200 7100
+	0    1    1    0
+$EndComp
+Wire Wire Line
+	1200 6950 1850 6950
+Wire Wire Line
+	1850 6950 1850 7250
+$Comp
+L power:GND #PWR0102
+U 1 1 5F8E247A
+P 800 7100
+F 0 "#PWR0102" H 800 6850 50  0001 C CNN
+F 1 "GND" V 805 6972 50  0000 R CNN
+F 2 "" H 800 7100 50  0001 C CNN
+F 3 "" H 800 7100 50  0001 C CNN
+	1    800  7100
+	0    1    1    0
+$EndComp
+Wire Wire Line
+	1000 7100 800  7100
+$Comp
+L power:GND #PWR0103
+U 1 1 5F8E2481
+P 1550 7100
+F 0 "#PWR0103" H 1550 6850 50  0001 C CNN
+F 1 "GND" V 1555 6972 50  0000 R CNN
+F 2 "" H 1550 7100 50  0001 C CNN
+F 3 "" H 1550 7100 50  0001 C CNN
+	1    1550 7100
+	0    -1   -1   0
+$EndComp
+Wire Wire Line
+	1400 7100 1550 7100
+$Comp
+L Device:R R2
+U 1 1 5F8E2488
+P 2050 7100
+F 0 "R2" H 2120 7146 50  0000 L CNN
+F 1 "10M" H 2120 7055 50  0000 L CNN
+F 2 "" V 1980 7100 50  0001 C CNN
+F 3 "~" H 2050 7100 50  0001 C CNN
+	1    2050 7100
+	1    0    0    -1
+$EndComp
+Wire Wire Line
+	2050 6950 1850 6950
+Connection ~ 1850 6950
+Wire Wire Line
+	2050 7250 1850 7250
+Connection ~ 1850 7250
+Wire Wire Line
+	2050 6950 2400 6950
+Connection ~ 2050 6950
+Wire Wire Line
+	2050 7250 2400 7250
+Connection ~ 2050 7250
+Wire Wire Line
+	1200 6950 1100 6950
+Wire Wire Line
+	800  6950 800  7100
+Connection ~ 1200 6950
+Connection ~ 800  7100
+Wire Wire Line
+	800  7100 800  7250
+$Comp
+L Device:C C17
+U 1 1 5F8E249B
+P 950 6950
+F 0 "C17" V 698 6950 50  0000 C CNN
+F 1 "C" V 789 6950 50  0000 C CNN
+F 2 "" H 988 6800 50  0001 C CNN
+F 3 "~" H 950 6950 50  0001 C CNN
+	1    950  6950
+	0    1    1    0
+$EndComp
+$Comp
+L Device:C C18
+U 1 1 5F8E24A1
+P 950 7250
+F 0 "C18" V 1250 7250 50  0000 C CNN
+F 1 "C" V 1150 7250 50  0000 C CNN
+F 2 "" H 988 7100 50  0001 C CNN
+F 3 "~" H 950 7250 50  0001 C CNN
+	1    950  7250
+	0    1    1    0
+$EndComp
+Connection ~ 1200 7250
+Wire Wire Line
+	1850 7250 1200 7250
+Wire Wire Line
+	1100 7250 1200 7250
+Text Label 2450 6050 0    50   ~ 0
+RTCX1
+Text Label 2450 6350 0    50   ~ 0
+RTCX2
+Text Label 2400 6950 0    50   ~ 0
+XTAL2
+Text Label 2400 7250 0    50   ~ 0
+XTAL1
+NoConn ~ 1050 6200
+NoConn ~ 1450 6200
+Wire Wire Line
+	2850 1400 2850 1550
+Wire Wire Line
+	2750 1400 2750 1550
+Wire Wire Line
+	1400 2800 1400 2700
+Connection ~ 1400 2700
+Wire Wire Line
+	1400 2600 1400 2500
+Wire Wire Line
+	1400 2700 1400 2600
+Connection ~ 1400 2600
+Connection ~ 1400 2500
+$Comp
 L Micro-rescue:LPC4337JBD144-LPC4337JBD144 U?
 U 1 1 5F5DA26E
@@
 	0    1    1    0
 $EndComp
-$Comp
-L power:PWR_FLAG #FLG0101
-U 1 1 5FE22055
-P 1200 2900
-F 0 "#FLG0101" H 1200 2975 50  0001 C CNN
-F 1 "PWR_FLAG" H 1200 3073 50  0000 C CNN
-F 2 "" H 1200 2900 50  0001 C CNN
-F 3 "~" H 1200 2900 50  0001 C CNN
-	1    1200 2900
-	1    0    0    -1
-$EndComp
-Connection ~ 1200 2900
-NoConn ~ 3450 4250
+Wire Wire Line
+	2600 1400 2600 1550
+Wire Wire Line
+	2500 1400 2500 1550
+Text Label 2500 1400 1    50   ~ 0
+XTAL2
+Text Label 2600 1400 1    50   ~ 0
+XTAL1
+Text Label 2750 1400 1    50   ~ 0
+RTCX2
+Text Label 2850 1400 1    50   ~ 0
+RTCX1
 $EndSCHEMATC
